File: hardware/control_board/control_board.kicad_sch (KiCad schematic)
At the start: 32 parts, among them J1 SWD, J2 Aux, J3 Panel, SW1 Reset, U1 STM32F103C8T6, Y1 8MHz

Commit message: Tidy up vias
Other:
- moved on the sheet: J2, R6, R7

Commit message: Minor layout adjustments
Parts:
- FB1: value 600R@100MHz -> 470R@100MHz
Changed lines of the file:
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@@
       (effects (font (size 1.27 1.27)) (justify left))
     )
-    (property "Value" "600R@100MHz" (at 69.85 171.45 90)
+    (property "Value" "470R@100MHz" (at 69.85 171.45 90)
       (effects (font (size 1.27 1.27)) (justify right))
     )

Commit message: Cleanup the project
Parts:
- FB1: value 470R@100MHz -> 470R
Changed lines of the file:
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@@
       (effects (font (size 1.27 1.27)) (justify left))
     )
-    (property "Value" "470R@100MHz" (at 69.85 171.45 90)
+    (property "Value" "470R" (at 69.85 171.45 90)
       (effects (font (size 1.27 1.27)) (justify right))
     )
